File: Modules/CP3 mixer/CP3 mixer.kicad_pcb (KiCad board)
At the start: 2 copper layers, 103 x 128.5 mm, 71 parts, among them J1 EURO_PWR_2x5, J2 PJ301M-12, J3 PJ301M-12, J4 PJ301M-12, J5 PJ301M-12, J6 PJ301M-12, J7 PJ301M-12, J8 PJ301M-12, J9 PJ301M-12, Q1 2N3904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

Commit message: Updated some projects to the new Kicad 6 format
Updated some projects to the new Kicad 6 format, and ( for the CP3 mixer ) fixed some footprints etc that were broken by the update
Parts:
- added REF**: Eurorack LED hole with ring, Eurocad:Eurorack_LED_hole_with_ring, F.Cu at (37.8, 91.5)
Other:
- net class Default removed
- net class Power removed
