File: Modules/Logic Neuron/Logic Neuron/Logic Neuron.sch (KiCad schematic (older format))
At the start: 87 parts, among them J1 PJ301M-12, J2 PJ301M-12, J3 PJ301M-12, J4 PJ301M-12, J5 PJ301M-12, J6 PJ301M-12, U1 TL074, U3 TL074, U4 TL074, U5 TL074, U6 TL074, U7 TL074, U8 TL074

Commit message: Logic neuron tweaks
- Fixed knob orientations
- Fixed polarity of stage 4 knob
- Fixed excessive atenuation at comparator inputs
Parts:
- added R? (x2): 100k, symbol Device:R
- added U?: TL074, symbol Amplifier_Operational:TL074
- R1: value 200k -> 100k
- R2: value 47k -> 10k
- R6, R7, R8: value 10k -> 100k
- RV1, RV2, RV3, RV4: symbol Device:R_POT -> eurocad:Potentiometer
- U1: value TL074 -> LM339
Connections:
- net -5V_regulated: now also R?.2; no longer J4.2
- net GND: now also U?.3 (+)
- net V_threshold: now also U1.11 (+), U1.5 (+), U1.7 (+); no longer U1.10 (-), U1.4 (-), U1.6 (-)
- net at D1.1 (K), R3.1, R6.2: now also U1.4 (-); no longer U1.5 (+)
- net at D2.1 (K), R4.1, R7.2: now also U1.6 (-); no longer U1.7 (+)
- net at D3.1 (K), R5.1, R8.2: now also U1.10 (-); no longer U1.11 (+)
- new net: R?.1, R?.2, U?.2 (-)
- new net +5V_ref: J4.2, R?.1, U?.1
Other:
- note added: "- Maybe just add another input for straight-through CV?\n- \n-Check the orientation of pots\n- check LED current\n- Check comparator is the correct way round\n- add voltage regulator\n- check comparator pinouts. ( opamps and comparators may be gotten switches somehow? )\n- Do we need to worry about offset voltage for the first opamps?"
- note added: "1.2V"
- note added: "Output between \n+1.5V ( pot CW )\n- 1.5V ( pot CCW )"
- note added: "When Input/2 > V_threshold, \ntransistor at output turns on"
- note added: "With +5V input:\n\n-Threshold goes between\n-5V ( pot CW )\n+5V ( pot CCW )\n\nSo +threshold goes between\n+5V ( power CW )\n- 5V ( pot CCW )"
- note removed: "-Check the orientation of pots\n- check LED current\n- Check comparator is the correct way round\n- add voltage regulator\n- check comparator pinouts. ( opamps and comparators may be gotten switches somehow? )"
- note removed: "Output between +-1.5V"
- note removed: "Output between +-5V\n\nCW = NEGATIVE output ( for +ve input )"
Changed lines of the file:
@@
 $EndDescr
 Text Notes 3525 950  0    50   ~ 0
--Check the orientation of pots\n- check LED current\n- Check comparator is the correct way round\n- add voltage regulator\n- check comparator pinouts. ( opamps and comparators may be gotten switches somehow? )
+- Maybe just add another input for straight-through CV?\n- \n-Check the orientation of pots\n- check LED current\n- Check comparator is the correct way round\n- add voltage regulator\n- check comparator pinouts. ( opamps and comparators may be gotten switches somehow? )\n- Do we need to worry about offset voltage for the first opamps?
 $Comp
 L Comparator:LM339 U1
@@
 P 2375 3525
 F 0 "U1" H 2333 3571 50  0000 L CNN
-F 1 "TL074" H 2333 3480 50  0000 L CNN
+F 1 "LM339" H 2333 3480 50  0000 L CNN
 F 2 "" H 2325 3625 50  0001 C CNN
 F 3 "https://www.st.com/resource/en/datasheet/lm139.pdf" H 2425 3725 50  0001 C CNN
@@
 P 875 3250
 F 0 "R1" H 945 3296 50  0000 L CNN
-F 1 "200k" H 945 3205 50  0000 L CNN
+F 1 "100k" H 945 3205 50  0000 L CNN
 F 2 "" V 805 3250 50  0001 C CNN
 F 3 "~" H 875 3250 50  0001 C CNN
@@
 P 875 3650
 F 0 "R2" H 945 3696 50  0000 L CNN
-F 1 "47k" H 945 3605 50  0000 L CNN
+F 1 "10k" H 945 3605 50  0000 L CNN
 F 2 "" V 805 3650 50  0001 C CNN
 F 3 "~" H 875 3650 50  0001 C CNN
@@
 Connection ~ 9425 3000
 $Comp
-L Device:R_POT RV2
+L eurocad:Potentiometer RV2
 U 1 1 61559C70
 P 8250 3100
@@
 Wire Notes Line
 	10100 2250 3725 2250
-Text Notes 9025 3325 0    50   ~ 0
-Output between +-1.5V
+Text Notes 9100 3425 0    50   ~ 0
+Output between \n+1.5V ( pot CW )\n- 1.5V ( pot CCW )
 $Comp
 L eurocad:PJ301M-12 J5
@@
 Connection ~ 7025 9875
 $Comp
-L Device:R_POT RV1
+L eurocad:Potentiometer RV1
 U 1 1 61638EC0
 P 5850 9975
@@
 Text GLabel 7150 9875 2    50   Input ~ 0
 -Threshold
-Text Notes 6500 10400 0    50   ~ 0
-Output between +-5V\n\nCW = NEGATIVE output ( for +ve input )
+Text Notes 6750 10775 0    50   ~ 0
+With +5V input:\n\n-Threshold goes between\n-5V ( pot CW )\n+5V ( pot CCW )\n\nSo +threshold goes between\n+5V ( power CW )\n- 5V ( pot CCW )
 Wire Wire Line
 	5225 9775 5850 9775
@@
 P 6700 3350
 F 0 "U1" H 6700 3175 50  0000 C CNN
-F 1 "TL074" H 6650 3350 50  0000 C CNN
+F 1 "LM339" H 6650 3350 50  0000 C CNN
 F 2 "" H 6650 3450 50  0001 C CNN
 F 3 "https://www.st.com/resource/en/datasheet/lm139.pdf" H 6750 3550 50  0001 C CNN
 	1    6700 3350
-	1    0    0    1
+	1    0    0    -1
 $EndComp
 Wire Wire Line
@@
 Wire Wire Line
 	2700 3525 2700 3625
-Wire Wire Line
-	5675 3450 5950 3450
-$Comp
-L Device:R R6
-U 1 1 6189D302
-P 5950 3700
-F 0 "R6" V 6125 3700 50  0000 C CNN
-F 1 "10k" V 6050 3700 50  0000 C CNN
-F 2 "" V 5880 3700 50  0001 C CNN
-F 3 "~" H 5950 3700 50  0001 C CNN
-	1    5950 3700
-	-1   0    0    1
-$EndComp
-Wire Wire Line
-	5950 3450 5950 3550
-Connection ~ 5950 3450
-Wire Wire Line
-	5950 3450 6225 3450
-$Comp
-L power:GND #PWR08
-U 1 1 618A3B26
-P 5950 3900
-F 0 "#PWR08" H 5950 3650 50  0001 C CNN
-F 1 "GND" V 5955 3772 50  0000 R CNN
-F 2 "" H 5950 3900 50  0001 C CNN
-F 3 "" H 5950 3900 50  0001 C CNN
-	1    5950 3900
-	1    0    0    -1
-$EndComp
-Wire Wire Line
-	5950 3850 5950 3900
 Text Notes 5675 8475 0    50   ~ 0
 Resistor grounds the signal\nif the input is left floating\n( eg unconnected wire )\n\nDiode ensures that the input doesn't go \nbelow the -ve rail of the comparator
@@
 Connection ~ 9450 4825
 $Comp
-L Device:R_POT RV3
+L eurocad:Potentiometer RV3
 U 1 1 6191F02A
 P 8275 4925
@@
 Wire Wire Line
 	7250 4725 7250 4675
-Text Notes 9050 5150 0    50   ~ 0
-Output between +-1.5V
 $Comp
 L Comparator:LM339 U1
@@
 P 6725 5175
 F 0 "U1" H 6725 5000 50  0000 C CNN
-F 1 "TL074" H 6675 5175 50  0000 C CNN
+F 1 "LM339" H 6675 5175 50  0000 C CNN
 F 2 "" H 6675 5275 50  0001 C CNN
 F 3 "https://www.st.com/resource/en/datasheet/lm139.pdf" H 6775 5375 50  0001 C CNN
 	2    6725 5175
-	1    0    0    1
-$EndComp
-Wire Wire Line
-	5700 5275 5975 5275
-$Comp
-L Device:R R7
-U 1 1 6191F04F
-P 5975 5525
-F 0 "R7" V 6150 5525 50  0000 C CNN
-F 1 "10k" V 6075 5525 50  0000 C CNN
-F 2 "" V 5905 5525 50  0001 C CNN
-F 3 "~" H 5975 5525 50  0001 C CNN
-	1    5975 5525
-	-1   0    0    1
-$EndComp
-Wire Wire Line
-	5975 5275 5975 5375
-Connection ~ 5975 5275
-Wire Wire Line
-	5975 5275 6250 5275
-$Comp
-L power:GND #PWR09
-U 1 1 6191F058
-P 5975 5725
-F 0 "#PWR09" H 5975 5475 50  0001 C CNN
-F 1 "GND" V 5980 5597 50  0000 R CNN
-F 2 "" H 5975 5725 50  0001 C CNN
-F 3 "" H 5975 5725 50  0001 C CNN
-	1    5975 5725
-	1    0    0    -1
-$EndComp
-Wire Wire Line
-	5975 5675 5975 5725
+	1    0    0    -1
+$EndComp
 $Comp
 L power:GND #PWR017
@@
 Connection ~ 9475 6650
 $Comp
-L Device:R_POT RV4
+L eurocad:Potentiometer RV4
 U 1 1 6193D731
 P 8300 6750
@@
 Wire Wire Line
 	7275 6550 7275 6500
-Text Notes 9075 6975 0    50   ~ 0
-Output between +-1.5V
-Wire Wire Line
-	5725 7100 6000 7100
-$Comp
-L Device:R R8
-U 1 1 6193D756
-P 6000 7350
-F 0 "R8" V 6175 7350 50  0000 C CNN
-F 1 "10k" V 6100 7350 50  0000 C CNN
-F 2 "" V 5930 7350 50  0001 C CNN
-F 3 "~" H 6000 7350 50  0001 C CNN
-	1    6000 7350
-	-1   0    0    1
-$EndComp
-Wire Wire Line
-	6000 7100 6000 7200
-Connection ~ 6000 7100
-Wire Wire Line
-	6000 7100 6275 7100
-$Comp
-L power:GND #PWR010
-U 1 1 6193D75F
-P 6000 7550
-F 0 "#PWR010" H 6000 7300 50  0001 C CNN
-F 1 "GND" V 6005 7422 50  0000 R CNN
-F 2 "" H 6000 7550 50  0001 C CNN
-F 3 "" H 6000 7550 50  0001 C CNN
-	1    6000 7550
-	1    0    0    -1
-$EndComp
-Wire Wire Line
-	6000 7500 6000 7550
 $Comp
 L power:GND #PWR018
@@
 F 3 "https://www.st.com/resource/en/datasheet/lm139.pdf" H 6800 7200 50  0001 C CNN
 	3    6750 7000
-	1    0    0    1
+	1    0    0    -1
 $EndComp
 $Comp
@@
 Wire Wire Line
 	5225 9875 5475 9875
-Text GLabel 5050 10575 0    50   Input ~ 0
--5V_regulated
 Text GLabel 12525 7850 0    50   Input ~ 0
 -Threshold
@@
 Text Notes 12150 6450 0    50   ~ 0
 Possible advantages: \nGate out varies cleanly between 0V and 10V
+Text Notes 1375 3575 0    50   ~ 0
+1.2V
+Text Notes 5925 3175 0    50   ~ 0
+1.2V
+Wire Wire Line
+	6000 7500 6000 7550
+$Comp
+L power:GND #PWR010
+U 1 1 6193D75F
+P 6000 7550
+F 0 "#PWR010" H 6000 7300 50  0001 C CNN
+F 1 "GND" V 6005 7422 50  0000 R CNN
+F 2 "" H 6000 7550 50  0001 C CNN
+F 3 "" H 6000 7550 50  0001 C CNN
+	1    6000 7550
+	1    0    0    -1
+$EndComp
+Wire Wire Line
+	6000 7100 6275 7100
+Wire Wire Line
+	5725 7100 6000 7100
+Connection ~ 6000 7100
+Wire Wire Line
+	6000 7100 6000 7200
+$Comp
+L Device:R R8
+U 1 1 6193D756
+P 6000 7350
+F 0 "R8" V 6175 7350 50  0000 C CNN
+F 1 "100k" V 6100 7350 50  0000 C CNN
+F 2 "" V 5930 7350 50  0001 C CNN
+F 3 "~" H 6000 7350 50  0001 C CNN
+	1    6000 7350
+	-1   0    0    1
+$EndComp
+Wire Wire Line
+	5975 5675 5975 5725
+$Comp
+L power:GND #PWR09
+U 1 1 6191F058
+P 5975 5725
+F 0 "#PWR09" H 5975 5475 50  0001 C CNN
+F 1 "GND" V 5980 5597 50  0000 R CNN
+F 2 "" H 5975 5725 50  0001 C CNN
+F 3 "" H 5975 5725 50  0001 C CNN
+	1    5975 5725
+	1    0    0    -1
+$EndComp
+Wire Wire Line
+	5975 5275 6250 5275
+Wire Wire Line
+	5700 5275 5975 5275
+Connection ~ 5975 5275
+Wire Wire Line
+	5975 5275 5975 5375
+$Comp
+L Device:R R7
+U 1 1 6191F04F
+P 5975 5525
+F 0 "R7" V 6150 5525 50  0000 C CNN
+F 1 "100k" V 6075 5525 50  0000 C CNN
+F 2 "" V 5905 5525 50  0001 C CNN
+F 3 "~" H 5975 5525 50  0001 C CNN
+	1    5975 5525
+	-1   0    0    1
+$EndComp
+Wire Wire Line
+	5950 3450 6225 3450
+Wire Wire Line
+	5675 3450 5950 3450
+Connection ~ 5950 3450
+Wire Wire Line
+	5950 3450 5950 3550
+Wire Wire Line
+	5950 3850 5950 3900
+$Comp
+L power:GND #PWR08
+U 1 1 618A3B26
+P 5950 3900
+F 0 "#PWR08" H 5950 3650 50  0001 C CNN
+F 1 "GND" V 5955 3772 50  0000 R CNN
+F 2 "" H 5950 3900 50  0001 C CNN
+F 3 "" H 5950 3900 50  0001 C CNN
+	1    5950 3900
+	1    0    0    -1
+$EndComp
+$Comp
+L Device:R R6
+U 1 1 6189D302
+P 5950 3700
+F 0 "R6" V 6125 3700 50  0000 C CNN
+F 1 "100k" V 6050 3700 50  0000 C CNN
+F 2 "" V 5880 3700 50  0001 C CNN
+F 3 "~" H 5950 3700 50  0001 C CNN
+	1    5950 3700
+	-1   0    0    1
+$EndComp
+Text Notes 6525 3800 0    50   ~ 0
+When Input/2 > V_threshold, \ntransistor at output turns on
+Text Notes 9225 5225 0    50   ~ 0
+Output between \n+1.5V ( pot CW )\n- 1.5V ( pot CCW )
+Text Notes 9225 7075 0    50   ~ 0
+Output between \n+1.5V ( pot CW )\n- 1.5V ( pot CCW )
+$Comp
+L Amplifier_Operational:TL074 U?
+U 1 1 615C6B91
+P 2400 5725
+F 0 "U?" H 2450 5575 50  0000 C CNN
+F 1 "TL074" H 2375 5725 50  0000 C CNN
+F 2 "" H 2350 5825 50  0001 C CNN
+F 3 "https://www.st.com/resource/en/datasheet/lm139.pdf" H 2450 5925 50  0001 C CNN
+	1    2400 5725
+	1    0    0    1
+$EndComp
+$Comp
+L power:GND #PWR?
+U 1 1 615C6B97
+P 2000 5925
+F 0 "#PWR?" H 2000 5675 50  0001 C CNN
+F 1 "GND" V 2005 5797 50  0000 R CNN
+F 2 "" H 2000 5925 50  0001 C CNN
+F 3 "" H 2000 5925 50  0001 C CNN
+	1    2000 5925
+	1    0    0    -1
+$EndComp
+Wire Wire Line
+	2100 5825 2000 5825
+Wire Wire Line
+	2000 5825 2000 5925
+$Comp
+L Device:R R?
+U 1 1 615C6B9F
+P 2475 5375
+F 0 "R?" V 2400 5375 50  0000 C CNN
+F 1 "100k" V 2475 5375 50  0000 C CNN
+F 2 "" V 2405 5375 50  0001 C CNN
+F 3 "~" H 2475 5375 50  0001 C CNN
+	1    2475 5375
+	0    1    1    0
+$EndComp
+Wire Wire Line
+	2325 5375 2050 5375
+Wire Wire Line
+	2625 5375 2800 5375
+$Comp
+L Device:R R?
+U 1 1 615C6BB1
+P 1825 5625
+F 0 "R?" V 1925 5625 50  0000 C CNN
+F 1 "100k" V 1825 5625 50  0000 C CNN
+F 2 "" V 1755 5625 50  0001 C CNN
+F 3 "~" H 1825 5625 50  0001 C CNN
+	1    1825 5625
+	0    1    1    0
+$EndComp
+Wire Wire Line
+	2700 5725 2800 5725
+Wire Wire Line
+	1975 5625 2050 5625
+Wire Wire Line
+	2050 5375 2050 5625
+Connection ~ 2050 5625
+Wire Wire Line
+	2050 5625 2100 5625
+Wire Wire Line
+	2800 5375 2800 5725
+Connection ~ 2800 5725
+Wire Wire Line
+	2800 5725 2900 5725
+Text GLabel 2900 5725 2    50   Input ~ 0
++5V_ref
+Text GLabel 1675 5625 0    50   Input ~ 0
+-5V_regulated
+Text GLabel 5050 10575 0    50   Input ~ 0
++5V_ref
 $EndSCHEMATC

Commit message: Logic neuron schematic update
Finalized most aspects: just need to assign opamp blocks, and opamp power
Parts:
- removed C3, C4: C_Small, symbol Device:C_Small
- removed C5, C6, C?: 10p, symbol Device:C_Small
- removed D? (x3): D, symbol Device:D
- removed D?: LED_Small, symbol Device:LED_Small
- removed J4, J6, J? (x4): PJ301M-12, symbol eurocad:PJ301M-12
- removed R12, R14: 4.7k, symbol Device:R
- removed R13, R15, R? (x2): 10k, symbol Device:R
- removed R16, R26, R27, R29, R30, R31, R32, R9, R? (x5): 100k, symbol Device:R
- removed R28: 91k, symbol Device:R
- removed R33: 470k, symbol Device:R
- removed R34, R35, R? (x4): 1k, symbol Device:R
- removed R?: 47k, symbol Device:R
- removed R?: R, symbol Device:R
- removed RV1: 100k, symbol eurocad:Potentiometer
- removed RV5: 20k, symbol Device:R_POT_TRIM
- removed unit 1 of U3
- removed U6, U7, U8, U? (x2): TL074, symbol Amplifier_Operational:TL074
- removed U?: LM339, symbol Comparator:LM339
- added C? (x2): 10p, symbol Device:C_Small
- added C? (x2): 100uF, symbol Device:CP1
- added C?: 100n, symbol Device:C
- added C?: 1uF, symbol Device:CP1
- added D?: D, symbol Device:D
- added D? (x4): LED, symbol Device:LED
- added D? (x2): 1N4001, Diode_THT:D_DO-41_SOD81_P10.16mm_Horizontal, symbol Diode:1N4001
- added D? (x2): LED_Bicolor_Tayda_A-1076, symbol eurocad:LED_Bicolor_Tayda_A-1076
- added F? (x2): Fuse 250mA (A-1391), symbol Device:Polyfuse_Small
- added J? (x4): PJ301M-12, symbol eurocad:PJ301M-12
- added J?: EURO_PWR_2x5, symbol eurocad:EURO_PWR_2x5
- added J? (x2): Conn_01x04, symbol Connector_Generic:Conn_01x04
- added R? (x5): 100k, symbol Device:R
- added R?: 91k, symbol Device:R
- added R?: 10k (RL), symbol Device:R
- added R? (x3): 3.3k, symbol Device:R
- added R? (x3): 1k, symbol Device:R
- added R?: 4.7k, symbol Device:R
- added R? (x3): 4.7k (RL), symbol Device:R
- added R? (x2): 10k, symbol Device:R
- added R? (x2): 150k, symbol Device:R
- added R? (x2): 470R, symbol Device:R
- added RV?: 20k, symbol Device:R_POT_TRIM
- added RV?: 100k, symbol eurocad:Potentiometer
- added U? (x5): TL074, symbol Amplifier_Operational:TL074
- added U?: LM79L05_TO92, Package_TO_SOT_THT:TO-92_Inline, symbol Regulator_Linear:LM79L05_TO92
- R10: value 4.7k -> 3.3k
- R2: value 10k -> 33k
Connections:
- net +12V: now also C?.1, D?.1 (K), F?.1; no longer R1.1
- net +5V_ref: now also R1.1, R?.1
- net -5V_regulated: now also C?.2, R?.2, U?.3 (VO)
- net GND: now also RV2.1, RV3.1, RV4.1, C?.1, C?.1, C?.1, C?.2, D?.1 (K), D?.1 (K), D?.2 (A), J?.1, J?.1, J?.1, J?.1, J?.1 (Pin_1), J?.1 (Pin_1), J?.2, J?.3 (GND), J?.4 (GND), J?.5 (GND), J?.6 (GND), J?.7 (GND), J?.8 (GND), R?.2, R?.2, R?.2, R?.2, R?.2, R?.2, R?.2, R?.2, R?.2, U?.1 (GND), U?.10 (+); no longer J1.2, J2.2, J3.2, RV2.3, RV3.3, RV4.3
- net at R11.1, U1.2: now also D?.1 (K)
- net at R10.1, R11.2, R17.1: now also RV2.3; no longer RV2.1
- net at R23.1, R24.1, R25.1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: now also C?.1, R?.1, R?.2
- net at U1.1: now also D?.1 (K), R?.1
- net at R18.1: now also RV3.3, R?.1, R?.2; no longer RV3.1
- net at U1.13: now also D?.1 (K), R?.1
- net at R19.1: now also RV4.3, R?.1, R?.2; no longer RV4.1
- net -SUM: no longer names the net of U5.1
- net -SUM: now also R?.2
- removed net Analog_1: R20.2, R21.2, R22.2, R23.2, U3.7, U3.8, U4.1
- net Analog_2 renamed -Analog_2
- net -Analog_2: now also R21.2, U3.7
- net Analog_3 renamed -Analog_3
- net -Analog_3: now also R22.2, U3.8
- net In1 renamed in1
- net in1: now also J?.2 (Pin_2)
- net In2 renamed in2
- net in2: now also J?.3 (Pin_3)
- net In3 renamed in3
- net in3: now also J?.4 (Pin_4)
- net Sum+Threshold renamed +SUM
- net +SUM: now also C?.2, J?.3, R?.1, R?.1, R?.1, U?.3 (+)
- new net: J?.3, R?.1
- new net: R?.2, R?.2, U?.9 (-)
- new net: D?.2 (A), U?.1
- new net: F?.2, J?.1 (+12V), J?.2 (+12V)
- new net: F?.2, J?.10 (-12V), J?.9 (-12V)
- new net: D?.1 (K), R?.2, R?.2
- new net: R?.1, RV?.3
- new net: D?.2 (A), R?.1 (x4)
- new net: R?.1, R?.1, U?.3 (+)
- new net: C?.2, R?.1, U?.1
- new net: C?.1, R?.1, U?.2 (-)
- new net: J?.3, J?.3, R?.2, R?.2
- new net: R?.2, RV?.3
- new net: R?.1, RV?.1
- new net: D?.2 (AK), U?.1 (x2)
- new net: D?.1 (KA), R?.1, U?.2 (-) (x2)
- new net: R?.1, R?.2, U?.3 (+)
- new net -12V: C?.2, C?.2, D?.2 (A), F?.1, U?.2 (VI)
- new net -Analog_1: R20.2, R23.2, U4.1
- new net -Analog_4: R?.2, RV?.1, RV?.2, U?.8
- new net Threshold: RV?.2, U?.2 (-), U?.3 (+)
- new net norm_in1: J1.2, J?.4 (Pin_4)
- new net norm_in2: J2.2, J?.3 (Pin_3)
- new net norm_in3: J3.2, J?.2 (Pin_2)
- no-connect marks 6 -> 4
Other:
- note added: "- check LED current\n- Check TL074 comparatoris the correct way round\n- check comparator pinouts. ( opamps and comparators may be gotten switches somehow? )\n- assign opamp blocks\n"
- note added: "-1.24V"
- note added: "Daisy chain input"
- note added: "Daisy chain output"
- note added: "LED indicators"
- note added: "Note: comparator\n-ve supply -5V"
- note added: "Output between \n-1.25V ( pot CW )\n+ 1.25V ( pot CCW )"
- note added: "This divider determines\nthe voltage of an "on" \ngate"
- note added: "Trim for accurate 1x amplification\n( input 4 to sum output )"
- note added: "try to put this opamp is on the same chip as the\nsumming opamp - the offset voltages may cancel (?)"
- note removed: "- Maybe just add another input for straight-through CV?\n- \n-Check the orientation of pots\n- check LED current\n- Check comparator is the correct way round\n- add voltage regulator\n- check comparator pinouts. ( opamps and comparators may be gotten switches somehow? )\n- Do we need to worry about offset voltage for the first opamps?"
- note removed: "-1.6V"
- note removed: "-SUM should be between +- 4.8V"
- note removed: "Assume LEDs require around 1mA"
- note removed: "Check orientation"
- note removed: "Check pot orientation"
- note removed: "Comparator output"
- note removed: "If SUM > THRESHOLD\n\nthen \n\n-THRESHOLD > -SUM"
- note removed: "Much simpler, and easier to incorporate LED\nBut the gate out level may be more variable? And there may be some crosstalk? Check.\nHow close will the "off" signal be to 0V?"
- note removed: "Notes:\n- The internal summing etc corresponds to the lower output level ( good for accurate CV control ): \n - Knobs 1-3 go from around -2V to 2V\n - Knob 4 ( with norm input ) - range TBD\n - Knob 4 ( with CV input ) is replicated reasonably precisely at the output when knob is fully CW\n\n- For the "high" output option, everything is scaled up 5x, so then knobs correpond to +- 7.5V. Better for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"
- note removed: "OPTION 1"
- note removed: "OPTION 2"
- note removed: "Output between \n+1.5V ( pot CW )\n- 1.5V ( pot CCW )"
- note removed: "Possible advantages: \nGate out varies cleanly between 0V and 10V"
- note removed: "Stages 1-3"
- note removed: "Using a regulated -ve rail \nfor the comparator, because\nit is being used as a reference\nfor the attenuverter knob\nand I would like it to be usable\nfor CV"
- note removed: "We need to do some ugly voltage clamping here, because the \ncomparator inputs must not see anything below -5V"
- note removed: "With +5V input:\n\n-Threshold goes between\n-5V ( pot CW )\n+5V ( pot CCW )\n\nSo +threshold goes between\n+5V ( power CW )\n- 5V ( pot CCW )"
- moved on the sheet: C1, C2, D1, D2, D3, J1, J2, J3, J5, R1, R10, R11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
