File: Modules/Logic Neuron/Logic Neuron/Logic Neuron.sch (KiCad schematic (older format))
At the start: 93 parts, among them J1 PJ301M-12, J2 PJ301M-12, J3 PJ301M-12, J5 PJ301M-12, U1 LM339, U3 TL074, U4 TL074, U5 TL074

Commit message: Updated some projects to the new Kicad 6 format
Updated some projects to the new Kicad 6 format, and ( for the CP3 mixer ) fixed some footprints etc that were broken by the update
Parts:
- removed C?: 1uF, symbol Device:CP1
- removed D1, D2, D3, D?: D, symbol Device:D
- removed U? (x5): TL074, symbol Amplifier_Operational:TL074
- added C10, C11, C12, C13, C14, C9: 100n, Eurocad:C_0805_2012Metric_Pad1.15x1.40mm_HandSolder_SmallTxt, symbol Device:C_Small
- added D1, D2, D3, D7: LL4148, Diode_SMD:D_MiniMELF, symbol Diode:LL4148
- added R47, R48, R7, R8: 100k, Eurocad:R_0805_2012Metric_Pad1.15x1.40mm_HandSolder_smallText, symbol Device:R
- added unit 4 of U1
- added unit 5 of U1
- added unit 4 of U2
- added unit 3 of U3
- added unit 4 of U3
- added unit 5 of U3
- added U4: TL074, Package_SO:SOIC-14_3.9x8.7mm_P1.27mm, symbol Amplifier_Operational:TL074
- C1, C2, C6: renamed from C?; footprint (none) -> Eurocad:C_0805_2012Metric_Pad1.15x1.40mm_HandSolder_SmallTxt
- C3, C4: renamed from C?; value 100uF -> 10uF; footprint (none) -> Capacitor_THT:CP_Radial_D5.0mm_P2.00mm
- C7: renamed from C1; footprint (none) -> Eurocad:C_0805_2012Metric_Pad1.15x1.40mm_HandSolder_SmallTxt
- C8: renamed from C2; footprint (none) -> Eurocad:C_0805_2012Metric_Pad1.15x1.40mm_HandSolder_SmallTxt
- D10, D9: renamed from D?; footprint (none) -> Eurocad:TaydaA-1076_bicolor_LED
- D4, D5, D6, D8: renamed from D?; footprint (none) -> Eurocad:LED3mm
- F1, F2: renamed from F?; footprint (none) -> Capacitor_THT:C_Disc_D7.5mm_W2.5mm_P5.00mm
- J1, J2, J3: footprint (none) -> Eurocad:PJ301M-12_Compact
- J10, J4, J8, J9: renamed from J?; footprint (none) -> Eurocad:PJ301M-12_Compact
- J11: renamed from J?; footprint (none) -> Eurocad:Eurorack_power_header
- J5, J6: renamed from J?; footprint (none) -> Connector_PinHeader_2.54mm:PinHeader_1x04_P2.54mm_Vertical
- J7: renamed from J5; footprint (none) -> Eurocad:PJ301M-12_Compact
- R1: renamed from R3; footprint (none) -> Eurocad:R_0805_2012Metric_Pad1.15x1.40mm_HandSolder_smallText
- R10, R16, R17, R18, R19, R29, R30, R31, R33, R34, R35, R36, R37, R38, R4, R40, R42, R45, R46: renamed from R?; footprint (none) -> Eurocad:R_0805_2012Metric_Pad1.15x1.40mm_HandSolder_smallText
- R11, R12, R13: renamed from R?; value 4.7k (RL) -> 1.5k (RL); footprint (none) -> Eurocad:R_0805_2012Metric_Pad1.15x1.40mm_HandSolder_smallText
- R14: renamed from R10; footprint (none) -> Eurocad:R_0805_2012Metric_Pad1.15x1.40mm_HandSolder_smallText
- R15: renamed from R11; footprint (none) -> Eurocad:R_0805_2012Metric_Pad1.15x1.40mm_HandSolder_smallText
- R2: renamed from R4; footprint (none) -> Eurocad:R_0805_2012Metric_Pad1.15x1.40mm_HandSolder_smallText
- R20: renamed from R17; footprint (none) -> Eurocad:R_0805_2012Metric_Pad1.15x1.40mm_HandSolder_smallText
- R21: renamed from R18; footprint (none) -> Eurocad:R_0805_2012Metric_Pad1.15x1.40mm_HandSolder_smallText
- R22: renamed from R19; footprint (none) -> Eurocad:R_0805_2012Metric_Pad1.15x1.40mm_HandSolder_smallText
- R23: renamed from R20; footprint (none) -> Eurocad:R_0805_2012Metric_Pad1.15x1.40mm_HandSolder_smallText
- R24: renamed from R21; footprint (none) -> Eurocad:R_0805_2012Metric_Pad1.15x1.40mm_HandSolder_smallText
- R25: renamed from R22; footprint (none) -> Eurocad:R_0805_2012Metric_Pad1.15x1.40mm_HandSolder_smallText
- R26: renamed from R23; footprint (none) -> Eurocad:R_0805_2012Metric_Pad1.15x1.40mm_HandSolder_smallText
- R27: renamed from R24; footprint (none) -> Eurocad:R_0805_2012Metric_Pad1.15x1.40mm_HandSolder_smallText
- R28: renamed from R25; footprint (none) -> Eurocad:R_0805_2012Metric_Pad1.15x1.40mm_HandSolder_smallText
- R3: renamed from R5; footprint (none) -> Eurocad:R_0805_2012Metric_Pad1.15x1.40mm_HandSolder_smallText
- R32: renamed from R?; value 10k (RL) -> 4.7k (RL); footprint (none) -> Eurocad:R_0805_2012Metric_Pad1.15x1.40mm_HandSolder_smallText
- R39, R41: renamed from R?; value 470R -> 660R; footprint (none) -> Eurocad:R_0805_2012Metric_Pad1.15x1.40mm_HandSolder_smallText
- R43: renamed from R1; footprint (none) -> Eurocad:R_0805_2012Metric_Pad1.15x1.40mm_HandSolder_smallText
- R44: renamed from R2; footprint (none) -> Eurocad:R_0805_2012Metric_Pad1.15x1.40mm_HandSolder_smallText
- R5: renamed from R6; footprint (none) -> Eurocad:R_0805_2012Metric_Pad1.15x1.40mm_HandSolder_smallText
- R6: renamed from R7; footprint (none) -> Eurocad:R_0805_2012Metric_Pad1.15x1.40mm_HandSolder_smallText
- R9: renamed from R8; footprint (none) -> Eurocad:R_0805_2012Metric_Pad1.15x1.40mm_HandSolder_smallText
- RV1: renamed from RV?; footprint (none) -> Potentiometer_THT:Potentiometer_Bourns_3296W_Vertical
- RV2, RV3, RV4: footprint (none) -> Eurocad:Alpha9mmPot
- RV5: renamed from RV?; footprint (none) -> Eurocad:Alpha9mmPot
- U1: renamed from U4; footprint (none) -> Package_SO:SOIC-14_3.9x8.7mm_P1.27mm
- U1: renamed from U3; footprint (none) -> Package_SO:SOIC-14_3.9x8.7mm_P1.27mm
- U2: renamed from U1; footprint (none) -> Package_SO:SOIC-14_3.9x8.7mm_P1.27mm
- U3: renamed from U5; footprint (none) -> Package_SO:SOIC-14_3.9x8.7mm_P1.27mm
- U3: renamed from U?; footprint (none) -> Package_SO:SOIC-14_3.9x8.7mm_P1.27mm
- U9: renamed from U?; value LM79L05_TO92 -> LM339; footprint Package_TO_SOT_THT:TO-92_Inline -> Package_SO:SOIC-14_3.9x8.7mm_P1.27mm
- gave numbers to parts that had none: 2
Connections:
- net +12V: now also C11.2, C13.2, C9.2, U1.4 (V+), U3.4 (V+), U4.4 (V+)
- net +5V_ref: now also U3.14
- net +SUM: now also U3.5 (+); no longer U3.3 (+)
- net -12V: now also C10.1, C12.1, C14.1, U1.11 (V-), U3.11 (V-), U4.11 (V-)
- net -Analog_4: now also U1.14
- net GND: now also C10.2, C11.1, C12.2, C13.1, C14.2, C9.1, D1.2 (A), D2.2 (A), D3.2 (A), R48.2, R7.1, R8.1, U1.12 (+), U3.12 (+), U4.10 (+), U4.12 (+)
- net Threshold: now also U3.6 (-), R47.1; no longer U3.2 (-)
- net at R1.1, R5.2, U2.4 (-): now also D1.1 (K)
- net at R45.1, R46.2: now also U3.13 (-)
- net at R10.2, R4.2: now also U1.13 (-)
- net at R32.2, R33.2: now also D7.1 (K)
- net at R33.1, R34.1: now also U3.10 (+)
- net at C2.2, R38.1: now also U3.8
- net at C2.1, R37.1: now also U3.9 (-)
- net at R2.1, R6.2, U2.6 (-): now also D2.1 (K)
- net gate_out: now reaches J10.3, J9.3, R37.2, R38.2
- net at R3.1, R9.2, U2.10 (-): now also D3.1 (K)
- net at D9.2 (AK): now also U4.1
- net at D9.1 (KA), R39.1: now also U4.2 (-)
- net at D10.2 (AK): now also U4.7
- net at D10.1 (KA), R41.1: now also U4.6 (-)
- net at R40.2, R42.1: now also U4.5 (+)
- new net: D7.2 (A), U3.7
- new net: R8.2, U2.8 (-)
- new net: R7.2, U2.9 (+)
- new net: R47.2, R48.1, U4.3 (+)
- new net: U4.8, U4.9 (-)
- new net: U4.13 (-), U4.14
- no-connect marks 4 -> 5
Other:
- note added: "Place this close \nto the 10uF caps!"
- note added: "Unused comparator"
- note added: "Unused opamps:\n[ why not use TL072? Because I have a big stash of TL074s, and TL074 is cheaper on Tayda ]\nSee https://www.analog.com/en/analog-dialogue/raqs/raq-issue-46.html"
- note added: "input stages"
- note added: "output stages"
- note added: "power"
- note added: "voltage references"
- note removed: "- check LED current\n- Check TL074 comparatoris the correct way round\n- check comparator pinouts. ( opamps and comparators may be gotten switches somehow? )\n- assign opamp blocks\n"
- moved on the sheet: C1, C2, C3, C4, C6, C7, C8, D10, D11, D12, D4, D5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
