File: Modules/Logic Neuron/Logic Neuron/Logic Neuron.kicad_sch (KiCad schematic)
At the start: 96 parts, among them J1 PJ301M-12, J10 PJ301M-12, J11 EURO_PWR_2x5, J2 PJ301M-12, J3 PJ301M-12, J4 PJ301M-12, J5 Conn_01x04, J6 Conn_01x04, J7 PJ301M-12, J8 PJ301M-12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

Commit message: Logic Neuron
Logic Neuron:
- Added LED indicator for input 4
- updated some footprints that were broken in the Kicad update
- started laying out the control board
Parts:
- removed U9: LM339, Package_SO:SOIC-14_3.9x8.7mm_P1.27mm, symbol Regulator_Linear:LM79L05_TO92
- added D13: LED_Bicolor_Tayda_A-1076, Eurocad:TaydaA-1076_bicolor_LED, symbol eurocad:LED_Bicolor_Tayda_A-1076
- added R49, R51: 100k, Eurocad:R_0805_2012Metric_Pad1.15x1.40mm_HandSolder_smallText, symbol Device:R
- added R50: 660R, Eurocad:R_0805_2012Metric_Pad1.15x1.40mm_HandSolder_smallText, symbol Device:R
- added U5: LM79L05_TO92, Package_TO_SOT_THT:TO-92_Inline, symbol Regulator_Linear:LM79L05_TO92
- C3, C4: symbol Device:CP1 -> Device:C_Polarized_Small
- D1, D2, D3, D7: footprint Diode_SMD:D_MiniMELF -> Eurocad:LL4148_sam
- RV1: symbol Device:R_POT_TRIM -> Device:R_Potentiometer_Trim
Connections:
- net -12V: now also U5.2 (VI)
- net -5V_regulated: now also U5.3 (VO)
- net -Analog_4: now also R49.1
- net GND: now also R50.2, R51.2, U5.1 (GND); no longer U4.10 (+)
- net LED_threshold: now reaches D9.2 (AK), U4.1
- net LED_SUM: now reaches D10.2 (AK), U4.7
- net at U4.9 (-): now also D13.2 (AK), R50.1; no longer U4.8
- new net: R49.2, R51.1, U4.10 (+)
- new net LED_in4: D13.1 (KA), U4.8
Other:
- moved on the sheet: R30, R31, R39, R40, R41, R42, R43, R44, R45, R46, R47, R48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

Commit message: Logic Neuron : PCB routing
Logic Neuron: First pass of PCB routing almost completed.

To do:
- ground planes
- DRCs
- silkscreen markings
Parts:
- added J12, J13: Conn_01x06, Connector_PinHeader_2.54mm:PinHeader_1x06_P2.54mm_Vertical, symbol Connector_Generic:Conn_01x06
- added J14, J15: Conn_01x08, Connector_PinHeader_2.54mm:PinHeader_1x08_P2.54mm_Vertical, symbol Connector_Generic:Conn_01x08
- added J16, J17: Conn_01x01, Connector_PinSocket_2.54mm:PinSocket_1x01_P2.54mm_Vertical, symbol Connector_Generic:Conn_01x01
- U5: footprint Package_TO_SOT_THT:TO-92_Inline -> Package_TO_SOT_THT:TO-92_HandSolder
Connections:
- net +12V: now also J14.6 (Pin_6), J15.6 (Pin_6)
- net -12V: now also J14.7 (Pin_7), J15.7 (Pin_7)
- net GND: now also U1.3 (+), J12.2 (Pin_2), J13.2 (Pin_2), J14.8 (Pin_8), J15.8 (Pin_8), J16.1 (Pin_1), J17.1 (Pin_1); no longer U1.12 (+)
- net Pot1: now also U1.12 (+); no longer U1.3 (+)
- net at R20.2, R23.1: now also U1.13 (-); no longer U1.2 (-)
- net at R45.1, R46.2: now also U1.2 (-); no longer U3.13 (-)
- net goutLED_b: now reaches R32.1
- net goutLED_b: now also J13.6 (Pin_6); no longer D8.2 (A)
- net +5V_ref renamed +5V_ref_f
- net +5V_ref_f: now also U1.1; no longer U3.14
- net +SUM renamed +SUM_b
- net +SUM_b: now also J13.4 (Pin_4); no longer J7.3, J8.3, R40.1
- net -5V_regulated renamed -5V_regulated_f
- net -5V_regulated_f: now also J14.5 (Pin_5); no longer C6.2, U5.3 (VO)
- removed net -Analog_1: R23.2, R26.2, U1.1
- net -Analog_2 renamed -Analog_2_f
- net -Analog_2_f: now also J14.2 (Pin_2); no longer R27.2
- net -Analog_3 renamed -Analog_3_f
- net -Analog_3_f: now also J14.3 (Pin_3); no longer R28.2
- net -Analog_4 renamed -Analog_4_b
- net -Analog_4_b: now also U3.14, J15.4 (Pin_4); no longer R49.1, U1.14
- net Threshold renamed Threshold_f
- net Threshold_f: now also J12.3 (Pin_3); no longer U3.6 (-)
- net V_threshold renamed V_threshold_f
- net gate_out renamed gout_b
- net gout_b: now also J13.5 (Pin_5); no longer J10.3, J9.3
- new net +SUM_f: J12.4 (Pin_4), J7.3, J8.3, R40.1
- new net -5V_regulated_b: C6.2, J15.5 (Pin_5), U5.3 (VO)
- new net -Analog_1_b: J15.1 (Pin_1), R26.2
- new net -Analog_1_f: J14.1 (Pin_1), R23.2, U1.14
- new net -Analog_2_b: J15.2 (Pin_2), R27.2
- new net -Analog_3_b: J15.3 (Pin_3), R28.2
- new net -Analog_4_f: J14.4 (Pin_4), R49.1
- new net Threshold_b: J13.3 (Pin_3), U3.6 (-)
- new net ch4_b: J13.1 (Pin_1), R10.2, U3.13 (-)
- new net ch4_f: J12.1 (Pin_1), R4.2
- new net goutLED_f: D8.2 (A), J12.6 (Pin_6)
- new net gout_f: J10.3, J12.5 (Pin_5), J9.3
Other:
- note added: "Components on Rear board"
- note added: "This is to help connect the birds together firmly"
- note added: "bottom of board"
- note added: "put this opamp is on the same chip as the summing opamp in the ope thaat offset voltages may cancel (?)"
- note added: "top of board"
- note removed: "try to put this opamp is on the same chip as the summing opamp - the offset voltages may cancel (?)"
- moved on the sheet: D8, J10, J5, J6, J7, J8, J9, R10, R4, RV1, U1A, U1D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
